File: kicad/leds/leds.kicad_pcb (KiCad board)
At the start: 2 copper layers, 16.5 x 44.5 mm, 11 parts, among them J1 Conn_01x04

Commit message: Tidy-ups pre-order
Parts:
- added REF**: OSHW-Logo2_9.8x8mm_SilkScreen, Symbol:OSHW-Logo2_9.8x8mm_SilkScreen, F.Cu at (119.4, 87.6)
Other:
- board text added: "Audio Lighting LEDs v1.0 Damian Moore 2020"
